Commit message: add ros__parameters namespace for vehicle_info.yaml.
Signed-off-by: Takamasa Horibe <horibe.takamasa@gmail.com>

File: urdf/vehicle.xacro (robot description, xacro)
@@ -6,5 +6,5 @@
   <link name="base_link">
     <visual>
-      <origin xyz="${vehicle_info['wheel_base']/2.0} 0 0" rpy="${pi/2.0} 0 ${pi}"/>
+      <origin xyz="${vehicle_info['/**']['ros__parameters']['wheel_base']/2.0} 0 0" rpy="${pi/2.0} 0 ${pi}"/>
       <geometry>
         <mesh filename="package://lexus_description/mesh/lexus.dae" scale="1 1 1"/>

Commit message: fix param file name in xacro file
Signed-off-by: mitsudome-r <ryohsuke.mitsudome@tier4.jp>

File: urdf/vehicle.xacro (robot description, xacro)
@@ -2,5 +2,5 @@
 <robot xmlns:xacro="http://ros.org/wiki/xacro">
   <!-- load parameter -->
-  <xacro:property name="vehicle_info" value="${load_yaml('$(find lexus_description)/config/vehicle_info.yaml')}"/>
+  <xacro:property name="vehicle_info" value="${load_yaml('$(find lexus_description)/config/vehicle_info.param.yaml')}"/>
   <!-- vehicle body -->
   <link name="base_link">
